Commit message: try to import mid360 but fail

File: src/world_models/models/simple_robot/robot.urdf (robot description, URDF)
Before this commit: robot simple_robot, 5 links, 4 joints
Links:
- removed link front_laser
- removed link left_laser
- removed link rear_laser
- removed link right_laser
- added link livox_mid360_link, mass 0.2; collision box size=0.08 0.08 0.05; visual box size=0.08 0.08 0.05
- link base_link: mass 10.0 -> 20.0; geometry collision box size=0.7 0.7 0.4; visual box size=0.7 0.7 0.4
Joints:
- removed joint front_laser_joint
- removed joint left_laser_joint
- removed joint rear_laser_joint
- removed joint right_laser_joint
- added joint livox_mid360_joint: type fixed, parent base_link, child livox_mid360_link, origin xyz=0 0 0.7 rpy=0 0 0
